Commit message: first commit

File: description/robot.urdf.xacro (robot description, xacro)
@@ -3,3 +3,5 @@
     <!-- Example link -->
     <xacro:include filename="robot_core.xacro"/>
+    <xacro:include filename="ros2_control.xacro"/>
+    <!-- <xacro:include filename="gazebo_control.xacro"/>  -->
 </robot>

File: description/robot_core.xacro (robot description, xacro)
@@ -42,4 +42,7 @@
         </xacro:inertial_box>
     </link>
+    <gazebo reference="chassis">
+        <material>Gazebo/White</material>
+    </gazebo>
     <!-- Left Wheel Link -->
     <joint name="left_wheel_joint" type="continuous">
@@ -66,4 +69,7 @@
         </xacro:inertial_cylinder>
     </link>
+    <gazebo reference="left_wheel">
+        <material>Gazebo/Blue</material>
+    </gazebo>
     <!-- Right Wheel Link -->
     <joint name="right_wheel_joint" type="continuous">
@@ -90,4 +96,7 @@
         </xacro:inertial_cylinder>
     </link>
+    <gazebo reference="right_wheel">
+        <material>Gazebo/Blue</material>
+    </gazebo>
     <!-- Caster Wheel Link -->
     <joint name="caster_wheel_joint" type="fixed">
@@ -113,3 +122,8 @@
         </xacro:inertial_sphere>
     </link>
+    <gazebo reference="caster_wheel">
+        <material>Gazebo/Black</material>
+        <mu1 value="0.001"/>
+        <mu2 value="0.001"/>
+    </gazebo>
 </robot>
